File: eda/dev/dev.kicad_pcb (KiCad board)
At the start: 2 copper layers, 0 parts

Commit message: development board finished
Parts:
- added C1: 0.1uF/100nF, 0_local:C_0603_1608Metric, F.Cu at (89.5, 98.8)
- added C2: 0.1uF/100nF, 0_local:C_0603_1608Metric, F.Cu at (94.0, 96.2)
- added D141: Blue, 0_local:LED_0603_1608Metric, F.Cu at (94.0, 118.2)
- added D142: Blue, 0_local:LED_0603_1608Metric, F.Cu at (92.0, 118.2)
- added D151: Yellow, 0_local:LED_0603_1608Metric, F.Cu at (116.5, 116.5)
- added D152: Yellow, 0_local:LED_0603_1608Metric, F.Cu at (116.5, 118.5)
- added D153: Yellow, 0_local:LED_0603_1608Metric, F.Cu at (116.5, 120.5)
- added D154: Yellow, 0_local:LED_0603_1608Metric, F.Cu at (116.5, 122.5)
- added D161: Blue, 0_local:LED_0603_1608Metric, F.Cu at (99.2, 118.2)
- added D162: Blue, 0_local:LED_0603_1608Metric, F.Cu at (97.2, 118.2)
- added D171: Blue, 0_local:LED_0603_1608Metric, F.Cu at (104.5, 118.2)
- added D172: Blue, 0_local:LED_0603_1608Metric, F.Cu at (102.5, 118.2)
- added D301: Yellow, 0_local:LED_0603_1608Metric, F.Cu at (116.5, 107.2)
- added D302: Yellow, 0_local:LED_0603_1608Metric, F.Cu at (116.5, 109.2)
- added D303: Yellow, 0_local:LED_0603_1608Metric, F.Cu at (116.5, 111.2)
- added D304: Yellow, 0_local:LED_0603_1608Metric, F.Cu at (116.5, 113.2)
- added D311: Red, 0_local:LED_0603_1608Metric, F.Cu at (116.5, 98.0)
- added D312: Red, 0_local:LED_0603_1608Metric, F.Cu at (116.5, 100.0)
- added D313: Red, 0_local:LED_0603_1608Metric, F.Cu at (116.5, 102.0)
- added D314: Red, 0_local:LED_0603_1608Metric, F.Cu at (116.5, 104.0)
- added D321: Blue, 0_local:LED_0603_1608Metric, F.Cu at (88.8, 118.2)
- added D322: Blue, 0_local:LED_0603_1608Metric, F.Cu at (86.8, 118.2)
- added D331: Red, 0_local:LED_0603_1608Metric, F.Cu at (116.5, 92.8)
- added D332: Red, 0_local:LED_0603_1608Metric, F.Cu at (116.5, 94.8)
- added D341: Red, 0_local:LED_0603_1608Metric, F.Cu at (116.5, 87.5)
- added D342: Red, 0_local:LED_0603_1608Metric, F.Cu at (116.5, 89.5)
- added G***: LOGO, 0_alt_bier:logo-alt_bier-1400dpi-7x16mm-front, F.Cu at (89.0, 86.5)
- added IC1: IC_CH552G, 0_local:IC_SOIC-16_3.9x9.9mm_Pitch1.27mm, F.Cu at (96.8, 101.8)
- added J1: USB_B_Micro, 0_local:USB_Micro-B_Jing, F.Cu at (78.5, 118.8)
- added J2: Conn_01x02, 0_local:Conn_Pin_Header_Straight_1x02_Pitch2.54mm, F.Cu at (79.0, 81.5)
- added R1: 10k Ohms, 0_local:R_0603_1608Metric, F.Cu at (77.8, 110.2)
- added R141: 220 Ohms, 0_local:R_0603_1608Metric, F.Cu at (94.0, 114.2)
- added R142: 220 Ohms, 0_local:R_0603_1608Metric, F.Cu at (92.0, 114.2)
- added R151: 220 Ohms, 0_local:R_0603_1608Metric, F.Cu at (112.5, 116.5)
- added R152: 220 Ohms, 0_local:R_0603_1608Metric, F.Cu at (112.5, 118.5)
- added R153: 220 Ohms, 0_local:R_0603_1608Metric, F.Cu at (112.5, 120.5)
- added R154: 220 Ohms, 0_local:R_0603_1608Metric, F.Cu at (112.5, 122.5)
- added R161: 220 Ohms, 0_local:R_0603_1608Metric, F.Cu at (99.2, 114.2)
- added R162: 220 Ohms, 0_local:R_0603_1608Metric, F.Cu at (97.2, 114.2)
- added R171: 220 Ohms, 0_local:R_0603_1608Metric, F.Cu at (104.5, 114.2)
- added R172: 220 Ohms, 0_local:R_0603_1608Metric, F.Cu at (102.5, 114.2)
- added R301: 220 Ohms, 0_local:R_0603_1608Metric, F.Cu at (112.5, 107.2)
- added R302: 220 Ohms, 0_local:R_0603_1608Metric, F.Cu at (112.5, 109.2)
- added R303: 220 Ohms, 0_local:R_0603_1608Metric, F.Cu at (112.5, 111.2)
- added R304: 220 Ohms, 0_local:R_0603_1608Metric, F.Cu at (112.5, 113.2)
- added R311: 220 Ohms, 0_local:R_0603_1608Metric, F.Cu at (112.5, 98.0)
- added R312: 220 Ohms, 0_local:R_0603_1608Metric, F.Cu at (112.5, 100.0)
- added R313: 220 Ohms, 0_local:R_0603_1608Metric, F.Cu at (112.5, 102.0)
- added R314: 220 Ohms, 0_local:R_0603_1608Metric, F.Cu at (112.5, 104.0)
- added R321: 220 Ohms, 0_local:R_0603_1608Metric, F.Cu at (88.8, 114.2)
- added R322: 220 Ohms, 0_local:R_0603_1608Metric, F.Cu at (86.8, 114.2)
- added R331: 220 Ohms, 0_local:R_0603_1608Metric, F.Cu at (112.5, 92.8)
- added R332: 220 Ohms, 0_local:R_0603_1608Metric, F.Cu at (112.5, 94.8)
- added R341: 220 Ohms, 0_local:R_0603_1608Metric, F.Cu at (112.5, 87.5)
- added R342: 220 Ohms, 0_local:R_0603_1608Metric, F.Cu at (112.5, 89.5)
- added S11: SW_TS2306A, 0_local:SW_TS2306A240GFMSM9_C388290, F.Cu at (104.8, 98.2)
- added SW1: SPDT_C136659, 0_local:SW_SPDT_PCM12_C136659, F.Cu at (78.2, 98.2)
- added SW2: TS2306A, 0_local:SW_TS2306A240GFMSM9_C388290, F.Cu at (81.8, 109.5)
Routing:
- net GND: track 0.00 -> 200.8 mm
- net D+: track 0.00 -> 40.6 mm
- net P1.5: track 0.00 -> 31.6 mm
- net D-: track 0.00 -> 29.1 mm
- net P3.1: track 0.00 -> 21.0 mm
- net P3.4: track 0.00 -> 20.4 mm
- net USB-PWR: track 0.00 -> 19.2 mm
- net V33: track 0.00 -> 18.6 mm
- net VCC: track 0.00 -> 18.2 mm
- net P3.0: track 0.00 -> 17.7 mm
- net P3.3: track 0.00 -> 17.0 mm
- net BAT-PWR: track 0.00 -> 14.2 mm
- net P1.7: track 0.00 -> 14.0 mm
- net P3.2: track 0.00 -> 12.5 mm
- net P1.6: track 0.00 -> 12.3 mm
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Other:
- board outline added: 48 x 48 mm
- board text added: "84Badge Development 0603 Components 84badge.com"
