File: eda/prod/prod.kicad_pcb (KiCad board)
At the start: 2 copper layers, 0 parts

Commit message: Started work on prod board
Parts:
- added C1: 0.1uF/100nF, 0_local:C_0603_1608Metric, F.Cu at (79.5, 129.2)
- added C2: 0.1uF/100nF, 0_local:C_0603_1608Metric, F.Cu at (79.3, 126.8)
- added D141: Blue, 0_local:LED_0603_1608Metric, F.Cu at (137.8, 162.8)
- added D142: Blue, 0_local:LED_0603_1608Metric, F.Cu at (143.0, 167.2)
- added D151: Yellow, 0_local:LED_0603_1608Metric, F.Cu at (137.5, 169.6)
- added D152: Yellow, 0_local:LED_0603_1608Metric, F.Cu at (150.3, 180.3)
- added D153: Yellow, 0_local:LED_0603_1608Metric, F.Cu at (129.7, 162.8)
- added D154: Yellow, 0_local:LED_0603_1608Metric, F.Cu at (147.1, 169.0)
- added D161: Blue, 0_local:LED_0603_1608Metric, F.Cu at (133.8, 162.8)
- added D162: Blue, 0_local:LED_0603_1608Metric, F.Cu at (129.7, 165.4)
- added D171: Blue, 0_local:LED_0603_1608Metric, F.Cu at (143.0, 171.3)
- added D172: Blue, 0_local:LED_0603_1608Metric, F.Cu at (140.6, 176.1)
- added D301: Yellow, 0_local:LED_0603_1608Metric, F.Cu at (132.2, 76.2)
- added D302: Yellow, 0_local:LED_0603_1608Metric, F.Cu at (138.0, 79.2)
- added D303: Yellow, 0_local:LED_0603_1608Metric, F.Cu at (145.5, 82.0)
- added D304: Yellow, 0_local:LED_0603_1608Metric, F.Cu at (152.8, 83.5)
- added D311: Red, 0_local:LED_0603_1608Metric, F.Cu at (146.3, 180.3)
- added D312: Red, 0_local:LED_0603_1608Metric, F.Cu at (147.1, 171.6)
- added D313: Red, 0_local:LED_0603_1608Metric, F.Cu at (144.7, 174.2)
- added D314: Red, 0_local:LED_0603_1608Metric, F.Cu at (133.5, 169.6)
- added D321: Blue, 0_local:LED_0603_1608Metric, F.Cu at (137.5, 167.0)
- added D322: Blue, 0_local:LED_0603_1608Metric, F.Cu at (144.7, 176.8)
- added D331: Red, 0_local:LED_0603_1608Metric, F.Cu at (134.5, 152.0)
- added D332: Red, 0_local:LED_0603_1608Metric, F.Cu at (134.5, 155.2)
- added D341: Red, 0_local:LED_0603_1608Metric, F.Cu at (141.8, 162.5)
- added D342: Red, 0_local:LED_0603_1608Metric, F.Cu at (148.7, 174.2)
- added G***: LOGO, 0_local:84_Badge_Silk_920dpi_127mm, F.Cu at (142.0, 83.2)
- added IC1: IC_CH552G, 0_local:IC_SOIC-16_3.9x9.9mm_Pitch1.27mm, F.Cu at (88.2, 125.0)
- added J1: USB_B_Micro, 0_local:USB_Micro-B_Jing, F.Cu at (101.5, 142.5)
- added J2: Conn_01x02, 0_local:Conn_Pin_Header_Straight_1x02_Pitch2.54mm, F.Cu at (80.0, 143.5)
- added R1: 10k Ohms, 0_local:R_0603_1608Metric, F.Cu at (72.8, 178.2)
- added R141: 220 Ohms, 0_local:R_0603_1608Metric, F.Cu at (100.8, 128.5)
- added R142: 220 Ohms, 0_local:R_0603_1608Metric, F.Cu at (100.8, 127.0)
- added R151: 220 Ohms, 0_local:R_0603_1608Metric, F.Cu at (95.0, 131.5)
- added R152: 220 Ohms, 0_local:R_0603_1608Metric, F.Cu at (95.0, 130.0)
- added R153: 220 Ohms, 0_local:R_0603_1608Metric, F.Cu at (95.0, 128.5)
- added R154: 220 Ohms, 0_local:R_0603_1608Metric, F.Cu at (95.0, 127.0)
- added R161: 220 Ohms, 0_local:R_0603_1608Metric, F.Cu at (95.0, 125.5)
- added R162: 220 Ohms, 0_local:R_0603_1608Metric, F.Cu at (95.0, 124.0)
- added R171: 220 Ohms, 0_local:R_0603_1608Metric, F.Cu at (95.0, 122.5)
- added R172: 220 Ohms, 0_local:R_0603_1608Metric, F.Cu at (95.0, 121.0)
- added R301: 220 Ohms, 0_local:R_0603_1608Metric, F.Cu at (88.2, 115.8)
- added R302: 220 Ohms, 0_local:R_0603_1608Metric, F.Cu at (89.8, 115.8)
- added R303: 220 Ohms, 0_local:R_0603_1608Metric, F.Cu at (91.2, 115.8)
- added R304: 220 Ohms, 0_local:R_0603_1608Metric, F.Cu at (92.8, 115.8)
- added R311: 220 Ohms, 0_local:R_0603_1608Metric, F.Cu at (95.0, 119.5)
- added R312: 220 Ohms, 0_local:R_0603_1608Metric, F.Cu at (95.0, 118.0)
- added R313: 220 Ohms, 0_local:R_0603_1608Metric, F.Cu at (95.0, 116.5)
- added R314: 220 Ohms, 0_local:R_0603_1608Metric, F.Cu at (95.0, 115.0)
- added R321: 220 Ohms, 0_local:R_0603_1608Metric, F.Cu at (100.8, 131.5)
- added R322: 220 Ohms, 0_local:R_0603_1608Metric, F.Cu at (100.8, 130.0)
- added R331: 220 Ohms, 0_local:R_0603_1608Metric, F.Cu at (115.0, 166.8)
- added R332: 220 Ohms, 0_local:R_0603_1608Metric, F.Cu at (115.2, 170.0)
- added R341: 220 Ohms, 0_local:R_0603_1608Metric, F.Cu at (122.0, 168.0)
- added R342: 220 Ohms, 0_local:R_0603_1608Metric, F.Cu at (122.2, 171.0)
- added S11: SW_TS2306A, 0_local:SW_TS2306A240GFMSM9_C388290, F.Cu at (94.0, 164.2)
- added SW1: SPDT_C136659, 0_local:SW_SPDT_PCM12_C136659, F.Cu at (90.0, 143.2)
- added SW2: TS2306A, 0_local:SW_TS2306A240GFMSM9_C388290, F.Cu at (110.2, 142.1)
Routing:
- net Net-(D312-Pad2): track 0.00 -> 4.98 mm
- net P3.1: track 0.00 -> 4.50 mm
- net P3.0: track 0.00 -> 4.50 mm
- net P1.5: track 0.00 -> 4.50 mm
- net Net-(D313-Pad2): track 0.00 -> 3.15 mm
- net P3.2: track 0.00 -> 1.50 mm
- net P1.7: track 0.00 -> 1.50 mm
- net P1.6: track 0.00 -> 1.50 mm
- net P1.4: track 0.00 -> 1.50 mm
- net Net-(D314-Pad2): track 0.00 -> 1.44 mm

Commit message: Badge PCB layout work
Parts:
- D141, D142, D151, D152, D153, D154, D161, D162, D171, D172, D301, D302, D303, D304, D311, D312, D313, D314, D321, D322, D331, D332, D341, D342: footprint 0_local:LED_0603_1608Metric -> 0_local:LED_0603_1608Metric_lowsilk
- moved D311 115.0 mm to (147.1, 65.3), turned to 100 degrees
- moved D142 112.4 mm to (182.7, 62.1), turned to 46 degrees
- moved D152 111.2 mm to (125.0, 72.0), turned to 346 degrees
- moved D171 110.4 mm to (158.4, 62.0), turned to 30 degrees
- moved D141 108.9 mm to (166.7, 57.8), turned to 28 degrees
- moved D161 106.8 mm to (162.3, 59.9), turned to 28 degrees
- moved D162 105.1 mm to (174.7, 70.3), turned to 45 degrees
- moved D312 104.9 mm to (153.6, 67.0)
- moved D321 104.1 mm to (154.7, 64.3), turned to 32 degrees
- moved D151 103.4 mm to (113.5, 69.0), turned to 345 degrees
- moved D172 100.8 mm to (166.6, 78.7), turned to 45 degrees
- moved D341 96.6 mm to (149.4, 66.2)
- moved D331 92.0 mm to (144.8, 60.6)
- moved D322 90.4 mm to (158.1, 87.4), turned to 45 degrees
- moved D154 86.6 mm to (147.2, 82.4), turned to 344 degrees
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Routing:
- net GND: track 0.00 -> 96.2 mm, vias 0 -> 2
- net D+: track 0.00 -> 41.5 mm
- net D-: track 0.00 -> 32.3 mm
- net V33: track 0.00 -> 27.0 mm
- net VCC: track 0.00 -> 18.2 mm
- net USB-PWR: track 0.00 -> 16.3 mm
- net P3.3: track 0.00 -> 10.2 mm
- net P3.4: track 0.00 -> 10.1 mm
- net BAT-PWR: track 0.00 -> 8.31 mm
- net P1.5: track 4.50 -> 10.1 mm
- net P3.0: track 4.50 -> 9.74 mm
- net P3.1: track 4.50 -> 8.79 mm
- net P1.7: track 1.50 -> 5.43 mm
- net P3.2: track 1.50 -> 5.04 mm
- net P1.4: track 1.50 -> 4.88 mm
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
Commit message: More PCB Layout work
Parts:
- removed the G*** at (142.0, 83.2)
- added G***: LOGO, 0_local:84_Badge_Silk_900dpi_127mm, F.Cu at (141.5, 84.5)
- moved D322 34.4 mm to (182.2, 62.9), turned to 47 degrees
- moved R154 23.0 mm to (82.2, 115.7), turned to 90 degrees
- moved R153 22.5 mm to (83.7, 115.7), turned to 90 degrees
- moved R152 22.1 mm to (85.2, 115.7), turned to 90 degrees
- moved R151 22.0 mm to (86.7, 115.7), turned to 90 degrees
- moved D332 20.5 mm to (152.2, 89.5), turned to 90 degrees
- moved R332 20.3 mm to (102.5, 117.0), turned to 0 degrees
- moved R331 18.8 mm to (102.5, 115.5), turned to 0 degrees
- moved R341 17.5 mm to (102.5, 118.5), turned to 0 degrees
- moved R342 16.4 mm to (102.5, 120.0), turned to 0 degrees
- moved D162 13.5 mm to (165.5, 80.2)
- moved D321 13.5 mm to (165.9, 56.9), turned to 30 degrees
- moved D172 13.1 mm to (157.7, 88.2)
- moved D142 13.0 mm to (173.7, 71.5)
- moved D313 8.21 mm to (156.6, 93.7)
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Routing:
- net GND: track 96.2 -> 617.8 mm, vias 2 -> 5
- net Net-(D321-Pad2): track 0.00 -> 179.7 mm
- net Net-(D141-Pad2): track 0.00 -> 173.1 mm
- net Net-(D322-Pad2): track 0.00 -> 160.6 mm
- net Net-(D142-Pad2): track 0.00 -> 154.0 mm
- net Net-(D161-Pad2): track 0.00 -> 153.0 mm
- net Net-(D171-Pad2): track 0.00 -> 148.0 mm
- net Net-(D162-Pad2): track 0.00 -> 128.0 mm
- net Net-(D154-Pad2): track 0.00 -> 122.3 mm
- net Net-(D172-Pad2): track 0.00 -> 121.5 mm
- net Net-(D312-Pad2): track 4.98 -> 124.1 mm
- net Net-(D311-Pad2): track 0.00 -> 118.4 mm
- net Net-(D153-Pad2): track 0.00 -> 109.5 mm
- net Net-(D331-Pad2): track 0.00 -> 101.1 mm
- net Net-(D341-Pad2): track 0.00 -> 100.3 mm
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- added copper zone on B.Cu, net GND
Other:
- board outline added: 130 x 120 mm
